File: switch_matrix.kicad_sch (KiCad schematic)
At the start: 0 parts

Commit message: switch matrix set-up
Parts:
- added D1, D10, D11, D12, D13, D14, D15, D16, D17, D18, D19, D2, D20, D21, D22, D23, D24, D25, D26, D27, D28, D29, D3, D30, D31, D32, D33, D34, D35, D36, D37, D38, D39, D4, D40, D41, D42, D43, D44, D45, D46, D47, D48, D49, D5, D50, D51, D52, D53, D54, D55, D56, D57, D58, D59, D6, D60, D61, D62, D63, D64, D65, D66, D67, D68, D69, D7, D70, D71, D72, D73, D74, D75, D76, D77, D78, D79, D8, D80, D81, D82, D83, D84, D85, D86, D87, D88, D89, D9, D90: 1N4148W, symbol Device:D
- added SW1, SW10, SW11, SW12, SW13, SW14, SW15, SW16, SW17, SW18, SW19, SW2, SW20, SW21, SW22, SW23, SW24, SW25, SW26, SW27, SW28, SW29, SW3, SW30, SW31, SW32, SW33, SW34, SW35, SW36, SW37, SW38, SW39, SW4, SW40, SW41, SW42, SW43, SW44, SW45, SW46, SW47, SW48, SW49, SW5, SW50, SW51, SW52, SW53, SW54, SW55, SW56, SW57, SW58, SW59, SW6, SW60, SW61, SW62, SW63, SW64, SW65, SW66, SW67, SW68, SW69, SW7, SW70, SW71, SW72, SW73, SW74, SW75, SW76, SW77, SW78, SW79, SW8, SW80, SW81, SW82, SW83, SW84, SW85, SW86, SW87, SW88, SW89, SW9, SW90: Kailh, symbol Switch:SW_Push
Connections:
- new net: D5.2 (A), SW5.1
- new net: D38.2 (A), SW38.1
- new net: D66.2 (A), SW66.1
- new net: D85.2 (A), SW85.1
- new net: D31.2 (A), SW31.1
- new net: D36.2 (A), SW36.1
- new net: D76.2 (A), SW76.1
- new net: D84.2 (A), SW84.1
- new net: D86.2 (A), SW86.1
- new net: D89.2 (A), SW89.1
- new net: D2.2 (A), SW2.1
- new net: D45.2 (A), SW45.1
- new net: D18.2 (A), SW18.1
- new net: D90.2 (A), SW90.1
- new net: D87.2 (A), SW87.1
- new net: D60.2 (A), SW60.1
- new net: D40.2 (A), SW40.1
- new net: D26.2 (A), SW26.1
- new net: D22.2 (A), SW22.1
- new net: D64.2 (A), SW64.1
- new net: D13.2 (A), SW13.1
- new net: D52.2 (A), SW52.1
- new net: D59.2 (A), SW59.1
- new net: D75.2 (A), SW75.1
- new net: D74.2 (A), SW74.1
- new net: D33.2 (A), SW33.1
- new net: D49.2 (A), SW49.1
- new net: D50.2 (A), SW50.1
- new net: D12.2 (A), SW12.1
- new net: D17.2 (A), SW17.1
- new net: D24.2 (A), SW24.1
- new net: D20.2 (A), SW20.1
- new net: D88.2 (A), SW88.1
- new net: D29.2 (A), SW29.1
- new net: D47.2 (A), SW47.1
- new net: D51.2 (A), SW51.1
- new net: D37.2 (A), SW37.1
- new net: D27.2 (A), SW27.1
- new net: D3.2 (A), SW3.1
- new net: D8.2 (A), SW8.1
- new net: D11.2 (A), SW11.1
- new net: D54.2 (A), SW54.1
- new net: D6.2 (A), SW6.1
- new net: D53.2 (A), SW53.1
- new net: D15.2 (A), SW15.1
- new net: D62.2 (A), SW62.1
- new net: D48.2 (A), SW48.1
- new net: D1.2 (A), SW1.1
- new net: D21.2 (A), SW21.1
- new net: D73.2 (A), SW73.1
- new net: D71.2 (A), SW71.1
- new net: D79.2 (A), SW79.1
- new net: D41.2 (A), SW41.1
- new net: D63.2 (A), SW63.1
- new net: D82.2 (A), SW82.1
- new net: D80.2 (A), SW80.1
- new net: D10.2 (A), SW10.1
- new net: D55.2 (A), SW55.1
- new net: D69.2 (A), SW69.1
- new net: D78.2 (A), SW78.1
- new net: D81.2 (A), SW81.1
- new net: D77.2 (A), SW77.1
- new net: D56.2 (A), SW56.1
- new net: D34.2 (A), SW34.1
- new net: D23.2 (A), SW23.1
- new net: D39.2 (A), SW39.1
- new net: D7.2 (A), SW7.1
- new net: D44.2 (A), SW44.1
- new net: D4.2 (A), SW4.1
- new net: D57.2 (A), SW57.1
- new net: D46.2 (A), SW46.1
- new net: D28.2 (A), SW28.1
- new net: D19.2 (A), SW19.1
- new net: D68.2 (A), SW68.1
- new net: D83.2 (A), SW83.1
- new net: D72.2 (A), SW72.1
- new net: D70.2 (A), SW70.1
- new net: D43.2 (A), SW43.1
- new net: D42.2 (A), SW42.1
- new net: D58.2 (A), SW58.1
- new net: D9.2 (A), SW9.1
- new net: D67.2 (A), SW67.1
- new net: D30.2 (A), SW30.1
- new net: D32.2 (A), SW32.1
- new net: D35.2 (A), SW35.1
- new net: D65.2 (A), SW65.1
- new net: D25.2 (A), SW25.1
- new net: D14.2 (A), SW14.1
- new net: D16.2 (A), SW16.1
- new net: D61.2 (A), SW61.1
- new net COL0: SW1.2, SW16.2, SW31.2, SW46.2, SW61.2, SW76.2
- new net COL1: SW17.2, SW2.2, SW32.2, SW47.2, SW62.2, SW77.2
- new net COL10: SW11.2, SW26.2, SW41.2, SW56.2, SW71.2, SW86.2
- new net COL11: SW12.2, SW27.2, SW42.2, SW57.2, SW72.2, SW87.2
- new net COL12: SW13.2, SW28.2, SW43.2, SW58.2, SW73.2, SW88.2
- new net COL13: SW14.2, SW29.2, SW44.2, SW59.2, SW74.2, SW89.2
- new net COL14: SW15.2, SW30.2, SW45.2, SW60.2, SW75.2, SW90.2
- new net COL2: SW18.2, SW3.2, SW33.2, SW48.2, SW63.2, SW78.2
- new net COL3: SW19.2, SW34.2, SW4.2, SW49.2, SW64.2, SW79.2
- new net COL4: SW20.2, SW35.2, SW5.2, SW50.2, SW65.2, SW80.2
- new net COL5: SW21.2, SW36.2, SW51.2, SW6.2, SW66.2, SW81.2
- new net COL6: SW22.2, SW37.2, SW52.2, SW67.2, SW7.2, SW82.2
- new net COL7: SW23.2, SW38.2, SW53.2, SW68.2, SW8.2, SW83.2
- new net COL8: SW24.2, SW39.2, SW54.2, SW69.2, SW84.2, SW9.2
- new net COL9: SW10.2, SW25.2, SW40.2, SW55.2, SW70.2, SW85.2
- new net ROW0: D1.1 (K), D10.1 (K), D11.1 (K), D12.1 (K), D13.1 (K), D14.1 (K), D15.1 (K), D2.1 (K), D3.1 (K), D4.1 (K), D5.1 (K), D6.1 (K), D7.1 (K), D8.1 (K), D9.1 (K)
- new net ROW1: D16.1 (K), D17.1 (K), D18.1 (K), D19.1 (K), D20.1 (K), D21.1 (K), D22.1 (K), D23.1 (K), D24.1 (K), D25.1 (K), D26.1 (K), D27.1 (K), D28.1 (K), D29.1 (K), D30.1 (K)
- new net ROW2: D31.1 (K), D32.1 (K), D33.1 (K), D34.1 (K), D35.1 (K), D36.1 (K), D37.1 (K), D38.1 (K), D39.1 (K), D40.1 (K), D41.1 (K), D42.1 (K), D43.1 (K), D44.1 (K), D45.1 (K)
- new net ROW3: D46.1 (K), D47.1 (K), D48.1 (K), D49.1 (K), D50.1 (K), D51.1 (K), D52.1 (K), D53.1 (K), D54.1 (K), D55.1 (K), D56.1 (K), D57.1 (K), D58.1 (K), D59.1 (K), D60.1 (K)
- new net ROW4: D61.1 (K), D62.1 (K), D63.1 (K), D64.1 (K), D65.1 (K), D66.1 (K), D67.1 (K), D68.1 (K), D69.1 (K), D70.1 (K), D71.1 (K), D72.1 (K), D73.1 (K), D74.1 (K), D75.1 (K)
- new net ROW5: D76.1 (K), D77.1 (K), D78.1 (K), D79.1 (K), D80.1 (K), D81.1 (K), D82.1 (K), D83.1 (K), D84.1 (K), D85.1 (K), D86.1 (K), D87.1 (K), D88.1 (K), D89.1 (K), D90.1 (K)

Commit message: documentation for switch matrix, peripherals
Other:
- note added: "6x15 Switch Matrix"
- title: (none) -> Switch Matrix
- moved on the sheet: D1, D10, D11, D12, D13, D14, D15, D16, D17, D18, D19, D2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
