File: rgb_leds.kicad_sch (KiCad schematic)
At the start: 0 parts

Commit message: finished LED daisychain
Parts:
- added C1, C10, C11, C12, C13, C14, C15, C16, C17, C18, C19, C2, C20, C21, C22, C23, C24, C25, C26, C27, C28, C29, C3, C30, C31, C32, C33, C34, C35, C36, C37, C38, C39, C4, C40, C41, C42, C43, C44, C45, C46, C47, C48, C49, C5, C50, C51, C52, C53, C54, C55, C56, C57, C58, C59, C6, C60, C61, C62, C63, C64, C65, C66, C67, C68, C69, C7, C70, C71, C72, C73, C74, C75, C76, C77, C78, C79, C8, C80, C81, C82, C83, C84, C85, C86, C9: 0.1uF, symbol Device:C
- added D1, D10, D11, D12, D13, D14, D15, D16, D17, D18, D19, D2, D20, D21, D22, D23, D24, D25, D26, D27, D28, D29, D3, D30, D31, D32, D33, D34, D35, D36, D37, D38, D39, D4, D40, D41, D42, D43, D44, D45, D46, D47, D48, D49, D5, D50, D51, D52, D53, D54, D55, D56, D57, D58, D59, D6, D60, D61, D62, D63, D64, D65, D66, D67, D68, D69, D7, D70, D71, D72, D73, D74, D75, D76, D77, D78, D79, D8, D80, D81, D82, D83, D84, D9: SK6812MINI-E, LED_SMD:LED_SK6812MINI-E_3.2x2.8mm_P1.5mm_ReverseMount, symbol LED:SK6812MINI-E
- added JP1, JP2: Open_Bridge, symbol Jumper:SolderJumper_3_Open
- added R1: 330, symbol Device:R
- added U1: TXU0101DBVR, SOT-23-6-DBV_TEX, symbol KeyboardSymbols:TXU0101DBVR
Connections:
- new net: D13.4 (DOUT), D14.2 (DIN)
- new net: D14.4 (DOUT), D15.2 (DIN)
- new net: D21.4 (DOUT), D22.2 (DIN)
- new net: D22.4 (DOUT), D23.2 (DIN)
- new net: D12.4 (DOUT), D13.2 (DIN)
- new net: D76.4 (DOUT), D77.2 (DIN)
- new net: D77.4 (DOUT), D78.2 (DIN)
- new net: D31.4 (DOUT), D32.2 (DIN)
- new net: D32.4 (DOUT), D33.2 (DIN)
- new net: D39.4 (DOUT), D40.2 (DIN)
- new net: D40.4 (DOUT), D41.2 (DIN)
- new net: D46.4 (DOUT), D47.2 (DIN)
- new net: D47.4 (DOUT), D48.2 (DIN)
- new net: D69.4 (DOUT), D70.2 (DIN)
- new net: D70.4 (DOUT), D71.2 (DIN)
- new net: D18.4 (DOUT), D19.2 (DIN)
- new net: D19.4 (DOUT), D20.2 (DIN)
- new net: D60.4 (DOUT), D61.2 (DIN)
- new net: D61.4 (DOUT), D62.2 (DIN)
- new net: D8.4 (DOUT), D9.2 (DIN)
- new net: D10.2 (DIN), D9.4 (DOUT)
- new net: D78.4 (DOUT), D79.2 (DIN)
- new net: D10.4 (DOUT), D11.2 (DIN)
- new net: D53.4 (DOUT), D54.2 (DIN)
- new net: D54.4 (DOUT), D55.2 (DIN)
- new net: D71.4 (DOUT), D72.2 (DIN)
- new net: D72.4 (DOUT), D73.2 (DIN)
- new net: D57.4 (DOUT), D58.2 (DIN)
- new net: D58.4 (DOUT), D59.2 (DIN)
- new net: D48.4 (DOUT), D49.2 (DIN)
- new net: D28.4 (DOUT), D29.2 (DIN)
- new net: D29.4 (DOUT), D30.2 (DIN)
- new net: D75.4 (DOUT), D76.2 (DIN)
- new net: D62.4 (DOUT), D63.2 (DIN)
- new net: D63.4 (DOUT), D64.2 (DIN)
- new net: D4.4 (DOUT), D5.2 (DIN)
- new net: D5.4 (DOUT), D6.2 (DIN)
- new net: D65.4 (DOUT), D66.2 (DIN)
- new net: D66.4 (DOUT), D67.2 (DIN)
- new net: D1.2 (DIN), R1.2
- new net: D1.4 (DOUT), D2.2 (DIN)
- new net: D50.4 (DOUT), D51.2 (DIN)
- new net: D51.4 (DOUT), D52.2 (DIN)
- new net: D82.4 (DOUT), D83.2 (DIN)
- new net: D83.4 (DOUT), D84.2 (DIN)
- new net: D15.4 (DOUT), D16.2 (DIN)
- new net: D56.4 (DOUT), D57.2 (DIN)
- new net: D25.4 (DOUT), D26.2 (DIN)
- new net: D26.4 (DOUT), D27.2 (DIN)
- new net: D59.4 (DOUT), D60.2 (DIN)
- new net: D7.4 (DOUT), D8.2 (DIN)
- new net: D11.4 (DOUT), D12.2 (DIN)
- new net: D20.4 (DOUT), D21.2 (DIN)
- new net: D27.4 (DOUT), D28.2 (DIN)
- new net: D38.4 (DOUT), D39.2 (DIN)
- new net: D64.4 (DOUT), D65.2 (DIN)
- new net: D2.4 (DOUT), D3.2 (DIN)
- new net: D3.4 (DOUT), D4.2 (DIN)
- new net: D81.4 (DOUT), D82.2 (DIN)
- new net: JP2.2 (C), R1.1
- new net: D80.4 (DOUT), D81.2 (DIN)
- new net: D37.4 (DOUT), D38.2 (DIN)
- new net: D16.4 (DOUT), D17.2 (DIN)
- new net: D17.4 (DOUT), D18.2 (DIN)
- new net: D73.4 (DOUT), D74.2 (DIN)
- new net: D30.4 (DOUT), D31.2 (DIN)
- new net: D6.4 (DOUT), D7.2 (DIN)
- new net: D67.4 (DOUT), D68.2 (DIN)
- new net: D24.4 (DOUT), D25.2 (DIN)
- new net: D23.4 (DOUT), D24.2 (DIN)
- new net: D49.4 (DOUT), D50.2 (DIN)
- new net: D74.4 (DOUT), D75.2 (DIN)
- new net: D55.4 (DOUT), D56.2 (DIN)
- new net: D41.4 (DOUT), D42.2 (DIN)
- new net: D42.4 (DOUT), D43.2 (DIN)
- new net: D68.4 (DOUT), D69.2 (DIN)
- new net: D44.4 (DOUT), D45.2 (DIN)
- new net: D45.4 (DOUT), D46.2 (DIN)
- new net: D43.4 (DOUT), D44.2 (DIN)
- new net: D36.4 (DOUT), D37.2 (DIN)
- new net: D79.4 (DOUT), D80.2 (DIN)
- new net: D33.4 (DOUT), D34.2 (DIN)
- new net: D52.4 (DOUT), D53.2 (DIN)
- new net: D35.4 (DOUT), D36.2 (DIN)
- new net: D34.4 (DOUT), D35.2 (DIN)
- new net +3.3V: C85.1, U1.1 (VCCA), U1.5 (OE)
- new net +5V: C1.1, C10.1, C11.1, C12.1, C13.1, C14.1, C15.1, C16.1, C17.1, C18.1, C19.1, C2.1, C20.1, C21.1, C22.1, C23.1, C24.1, C25.1, C26.1, C27.1, C28.1, C29.1, C3.1, C30.1, C31.1, C32.1, C33.1, C34.1, C35.1, C36.1, C37.1, C38.1, C39.1, C4.1, C40.1, C41.1, C42.1, C43.1, C44.1, C45.1, C46.1, C47.1, C48.1, C49.1, C5.1, C50.1, C51.1, C52.1, C53.1, C54.1, C55.1, C56.1, C57.1, C58.1, C59.1, C6.1, C60.1, C61.1, C62.1, C63.1, C64.1, C65.1, C66.1, C67.1, C68.1, C69.1, C7.1, C70.1, C71.1, C72.1, C73.1, C74.1, C75.1, C76.1, C77.1, C78.1, C79.1, C8.1, C80.1, C81.1, C82.1, C83.1, C84.1, C86.1, C9.1, D1.3 (VDD), D10.3 (VDD), D11.3 (VDD), D12.3 (VDD), D13.3 (VDD), D14.3 (VDD), D15.3 (VDD), D16.3 (VDD), D17.3 (VDD), D18.3 (VDD), D19.3 (VDD), D2.3 (VDD), D20.3 (VDD), D21.3 (VDD), D22.3 (VDD), D23.3 (VDD), D24.3 (VDD), D25.3 (VDD), D26.3 (VDD), D27.3 (VDD), D28.3 (VDD), D29.3 (VDD), D3.3 (VDD), D30.3 (VDD), D31.3 (VDD), D32.3 (VDD), D33.3 (VDD), D34.3 (VDD), D35.3 (VDD), D36.3 (VDD), D37.3 (VDD), D38.3 (VDD), D39.3 (VDD), D4.3 (VDD), D40.3 (VDD), D41.3 (VDD), D42.3 (VDD), D43.3 (VDD), D44.3 (VDD), D45.3 (VDD), D46.3 (VDD), D47.3 (VDD), D48.3 (VDD), D49.3 (VDD), D5.3 (VDD), D50.3 (VDD), D51.3 (VDD), D52.3 (VDD), D53.3 (VDD), D54.3 (VDD), D55.3 (VDD), D56.3 (VDD), D57.3 (VDD), D58.3 (VDD), D59.3 (VDD), D6.3 (VDD), D60.3 (VDD), D61.3 (VDD), D62.3 (VDD), D63.3 (VDD), D64.3 (VDD), D65.3 (VDD), D66.3 (VDD), D67.3 (VDD), D68.3 (VDD), D69.3 (VDD), D7.3 (VDD), D70.3 (VDD), D71.3 (VDD), D72.3 (VDD), D73.3 (VDD), D74.3 (VDD), D75.3 (VDD), D76.3 (VDD), D77.3 (VDD), D78.3 (VDD), D79.3 (VDD), D8.3 (VDD), D80.3 (VDD), D81.3 (VDD), D82.3 (VDD), D83.3 (VDD), D84.3 (VDD), D9.3 (VDD), U1.6 (VCCB)
- new net GND: C1.2, C10.2, C11.2, C12.2, C13.2, C14.2, C15.2, C16.2, C17.2, C18.2, C19.2, C2.2, C20.2, C21.2, C22.2, C23.2, C24.2, C25.2, C26.2, C27.2, C28.2, C29.2, C3.2, C30.2, C31.2, C32.2, C33.2, C34.2, C35.2, C36.2, C37.2, C38.2, C39.2, C4.2, C40.2, C41.2, C42.2, C43.2, C44.2, C45.2, C46.2, C47.2, C48.2, C49.2, C5.2, C50.2, C51.2, C52.2, C53.2, C54.2, C55.2, C56.2, C57.2, C58.2, C59.2, C6.2, C60.2, C61.2, C62.2, C63.2, C64.2, C65.2, C66.2, C67.2, C68.2, C69.2, C7.2, C70.2, C71.2, C72.2, C73.2, C74.2, C75.2, C76.2, C77.2, C78.2, C79.2, C8.2, C80.2, C81.2, C82.2, C83.2, C84.2, C85.2, C86.2, C9.2, D1.1 (VSS), D10.1 (VSS), D11.1 (VSS), D12.1 (VSS), D13.1 (VSS), D14.1 (VSS), D15.1 (VSS), D16.1 (VSS), D17.1 (VSS), D18.1 (VSS), D19.1 (VSS), D2.1 (VSS), D20.1 (VSS), D21.1 (VSS), D22.1 (VSS), D23.1 (VSS), D24.1 (VSS), D25.1 (VSS), D26.1 (VSS), D27.1 (VSS), D28.1 (VSS), D29.1 (VSS), D3.1 (VSS), D30.1 (VSS), D31.1 (VSS), D32.1 (VSS), D33.1 (VSS), D34.1 (VSS), D35.1 (VSS), D36.1 (VSS), D37.1 (VSS), D38.1 (VSS), D39.1 (VSS), D4.1 (VSS), D40.1 (VSS), D41.1 (VSS), D42.1 (VSS), D43.1 (VSS), D44.1 (VSS), D45.1 (VSS), D46.1 (VSS), D47.1 (VSS), D48.1 (VSS), D49.1 (VSS), D5.1 (VSS), D50.1 (VSS), D51.1 (VSS), D52.1 (VSS), D53.1 (VSS), D54.1 (VSS), D55.1 (VSS), D56.1 (VSS), D57.1 (VSS), D58.1 (VSS), D59.1 (VSS), D6.1 (VSS), D60.1 (VSS), D61.1 (VSS), D62.1 (VSS), D63.1 (VSS), D64.1 (VSS), D65.1 (VSS), D66.1 (VSS), D67.1 (VSS), D68.1 (VSS), D69.1 (VSS), D7.1 (VSS), D70.1 (VSS), D71.1 (VSS), D72.1 (VSS), D73.1 (VSS), D74.1 (VSS), D75.1 (VSS), D76.1 (VSS), D77.1 (VSS), D78.1 (VSS), D79.1 (VSS), D8.1 (VSS), D80.1 (VSS), D81.1 (VSS), D82.1 (VSS), D83.1 (VSS), D84.1 (VSS), D9.1 (VSS), U1.2 (GND)
- new net LED_DATA: JP1.2 (C)
- new net LED_DATA_LS_IN: JP1.3 (B), U1.3 (A)
- new net LED_DATA_LS_OUT: JP2.1 (A), U1.4 (BY)
- new net LED_DATA_RAW: JP1.1 (A), JP2.3 (B)
- no-connect marks 0 -> 1

Commit message: documentation for rgb sheet
Other:
- note added: "3.3V <-> 5V Level Shifter"
- note added: "BRIDGES and 330-OHM SERIES RESISTOR"
- note added: "Daisy-Chained SK6812 MINI-E RGB LEDs"
- moved on the sheet: C1, C10, C11, C12, C13, C14, C15, C16, C17, C18, C19, C2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
